Commit message: Corregit error en articulacio i creada plataforma

File: aibo_model/Aibo.urdf (robot description, URDF)
Before this commit: robot Aibo, 17 links, 16 joints
Joints:
- joint LB_down_leg_joint: origin xyz=-0 -0.009 -0.0375 rpy=-0.38025 0 0 -> xyz=0 -0.009 -0.065 rpy=-0.38025 0 0
- joint LB_up_leg_rot_x_joint: origin xyz=0 0 -0.0275 rpy=0 0 0 -> xyz=0 0 0 rpy=0 0 0
- joint LF_down_leg_joint: origin xyz=0 0.009 -0.0375 rpy=0.38025 0 0 -> xyz=0 0.009 -0.065 rpy=0.38025 0 0
- joint LF_up_leg_rot_x_joint: origin xyz=0 0 -0.0275 rpy=0 0 0 -> xyz=0 0 0 rpy=0 0 0
- joint RB_down_leg_joint: origin xyz=0 -0.009 -0.0375 rpy=-0.38025 0 0 -> xyz=0 -0.009 -0.065 rpy=-0.38025 0 0
- joint RB_up_leg_rot_x_joint: origin xyz=0 0 -0.0275 rpy=0 0 0 -> xyz=0 0 0 rpy=0 0 0
- joint RF_down_leg_joint: origin xyz=0 0.009 -0.0375 rpy=0.38025 0 0 -> xyz=0 0.009 -0.065 rpy=0.38025 0 0
- joint RF_up_leg_rot_x_joint: origin xyz=0 0 -0.0275 rpy=0 0 0 -> xyz=0 0 0 rpy=0 0 0
